File: KiCad/LNA_IN.kicad_sch (KiCad schematic)
At the start: 6 parts

Commit message: prepare to move barometer to front
Parts:
- AE1: now not fitted
Changed lines of the file:
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@@
 		(in_bom yes)
 		(on_board yes)
-		(dnp no)
+		(dnp yes)
 		(fields_autoplaced yes)
 		(property "Reference" "AE1"
