File: KiCad/PyroChannel.kicad_sch (KiCad schematic)
At the start: 5 parts, among them Q3 IRLML0030

Commit message: finalize board
Changed lines of the file:
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@@
 		(on_board yes)
 		(dnp no)
-		(fields_autoplaced yes)
 		(property "Reference" "Q3"
 			(at 151.13 92.7099 0)
@@
 		)
 		(property "LCSC" "C67272"
-			(at 144.78 93.98 0)
+			(at 146.304 93.726 0)
 			(effects
 				(font

Commit message: further refine board
Parts:
- R19: value 10k -> 5.1k; LCSC C25744 -> C25905
Changed lines of the file:
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@@
 		(fields_autoplaced yes)
 		(property "Reference" "R19"
-			(at 160.02 95.2499 0)
+			(at 160.02 93.9799 0)
 			(effects
 				(font
@@
 			)
 		)
-		(property "Value" "10k"
-			(at 160.02 97.7899 0)
+		(property "Value" "5.1k"
+			(at 160.02 96.5199 0)
 			(effects
 				(font
@@
 			)
 		)
-		(property "LCSC" "C25744"
-			(at 157.48 96.52 0)
+		(property "LCSC" "C25905"
+			(at 160.02 99.0599 0)
 			(effects
 				(font
 					(size 1.27 1.27)
 				)
+				(justify left)
 			)
 		)
